Commit message: New draft

File: rigby/urdf/rigby.urdf (robot description, URDF)
Before this commit: robot rigby, 40 links, 39 joints
Links:
- removed link Base
- removed link Lower_Arm
- removed link Rotation_Pitch
- removed link Upper_Arm
- removed link Wrist_Pitch_Roll
- added link right_arm_base_link, mass 0.147; collision mesh filename=meshes/base_motor_holder_so101_v1.stl; collision mesh filename=meshes/base_so101_v2.stl
- added link right_arm_lower_arm_link, mass 0.104; collision mesh filename=meshes/motor_holder_so101_wrist_v1.stl; collision mesh filename=meshes/sts3215_03a_v1.stl
- added link right_arm_shoulder_link, mass 0.100006; collision mesh filename=meshes/motor_holder_so101_base_v1.stl; collision mesh filename=meshes/rotation_pitch_so101_v1.stl
- added link right_arm_upper_arm_link, mass 0.103; collision mesh filename=meshes/sts3215_03a_v1.stl; collision mesh filename=meshes/upper_arm_so101_v1.stl
- added link right_arm_wrist_link, mass 0.079; collision mesh filename=meshes/sts3215_03a_no_horn_v1.stl; collision mesh filename=meshes/wrist_roll_pitch_so101_v2.stl
- link base_link: mass 70.1294 -> 11.534; geometry collision box size=0.009 0.405 0.09; collision box size=0.009 0.405 0.09
- link left_arm_Gripper_Jaw_01_v1_1: geometry collision box size=0.0040003 0.02706 0.03498; visual mesh filename=meshes/Gripper_Jaw_01_v1_1.stl scale=0.001 0.001 0.001
- link left_arm_Gripper_Jaw_02_v1_1: geometry collision box size=0.0040001 0.02706 0.03498; visual mesh filename=meshes/Gripper_Jaw_02_v1_1.stl scale=0.001 0.001 0.001
- link left_arm_ST3215_1_v1_1: mass 0.03190666159632515 -> 0.055
- link left_arm_ST3215_2_v1_1: mass 0.03190666159632515 -> 0.055
- link left_arm_ST3215_3_v1_1: mass 0.03190666159632515 -> 0.055
- link left_arm_ST3215_4_v1_1: mass 0.03190666159632515 -> 0.055
- link left_arm_ST3215_5_v1_1: mass 0.03190666159632515 -> 0.055
- link left_arm_ST3215_6_v1_1: mass 0.03190666159632515 -> 0.055
- link left_arm_ST3215_7_v1_1: mass 0.03190666159632515 -> 0.055
- link left_arm_ST3215_8_v1_1: mass 0.03190666159632515 -> 0.055
- link left_wrist_camera_link: geometry visual box size=0.012 0.025 0.025
- link right_arm_Gripper_Jaw_01_v1_1: geometry collision box size=0.0040003 0.02706 0.03498; visual mesh filename=meshes/Gripper_Jaw_01_v1_1.stl scale=0.001 0.001 0.001
- link right_arm_Gripper_Jaw_02_v1_1: geometry collision box size=0.0040001 0.02706 0.03498; visual mesh filename=meshes/Gripper_Jaw_02_v1_1.stl scale=0.001 0.001 0.001
- link right_arm_ST3215_8_v1_1: mass 0.03190666159632515 -> 0.055
- link right_wrist_camera_link: geometry visual box size=0.012 0.025 0.025
- link root_arm_1_link_1: mass 0 -> 0.001
- link root_arm_1_link_2: mass 0 -> 0.001
Joints:
- removed joint Elbow
- removed joint Pitch
- removed joint Rotation
- removed joint Wrist_Pitch
- removed joint Wrist_Roll
- removed joint arm_base_joint
- added joint right_arm_elbow_flex: type revolute, parent right_arm_upper_arm_link, child right_arm_lower_arm_link, origin xyz=-0.11257 -0.028 1.73763e-16 rpy=-3.63608e-16 8.74301e-16 1.5708, axis 0 0 1, limit lower=-1.69 upper=1.69 effort=10 velocity=10
- added joint right_arm_mount: type fixed, parent base_link, child right_arm_base_link, origin xyz=0.0713647 -0.133 0.7624 rpy=0 0 0
- added joint right_arm_shoulder_lift: type revolute, parent right_arm_shoulder_link, child right_arm_upper_arm_link, origin xyz=-0.0303992 -0.0182778 -0.0542 rpy=-1.5708 -1.5708 0, axis 0 0 1, limit lower=-1.74533 upper=1.74533 effort=10 velocity=10
- added joint right_arm_shoulder_pan: type revolute, parent right_arm_base_link, child right_arm_shoulder_link, origin xyz=0.0388353 -8.97657e-09 0.0624 rpy=3.14159 4.18253e-17 -3.14159, axis 0 0 1, limit lower=-1.91986 upper=1.91986 effort=10 velocity=10
- added joint right_arm_wrist_flex: type revolute, parent right_arm_lower_arm_link, child right_arm_wrist_link, origin xyz=-0.1349 0.0052 3.62355e-17 rpy=4.02456e-15 8.67362e-16 -1.5708, axis 0 0 1, limit lower=-1.65806 upper=1.65806 effort=10 velocity=10
- added joint right_arm_wrist_roll: type revolute, parent right_arm_wrist_link, child right_arm_Gripper_Base_v1_1, origin xyz=2.04446e-08 -0.0538817 0.0181 rpy=2.36618 1.54652 -0.784594, axis -0.017144 -0.999812 0.009029, limit lower=-2.74385 upper=2.84121 effort=10 velocity=10
- joint context_camera_1_aim_joint: origin xyz=0 0 0 rpy=2.02381 1.6581 1.85905 -> xyz=0 0 0 rpy=0 -0.03817 0.07854
- joint context_camera_1_joint: origin xyz=0.065286 -0.005502 1.014072 rpy=0 0.48869 0 -> xyz=0.079413 -0.005502 1.006560 rpy=0 0.48869 0
- joint context_camera_1_optical_joint: origin xyz=0 0 0 rpy=0 0 0.83103 -> xyz=0 0 0 rpy=-1.5708 0 -1.5708
- joint left_wrist_camera_joint: origin xyz=0.0 0.03 0.07 rpy=-0.45 1.5708 0 -> xyz=0.0 0.03 0.07 rpy=0 0.45 1.5708
- joint right_wrist_camera_joint: origin xyz=0.0 0.03 0.07 rpy=-0.45 1.5708 0 -> xyz=0.0 0.03 0.07 rpy=0 0.45 1.5708

Commit message: Further project carousel changes

File: rigby/urdf/rigby.urdf (robot description, URDF)
Before this commit: robot rigby, 40 links, 39 joints
Links:
- link base_link: geometry collision box size=0.009 0.405 0.09; collision box size=0.009 0.405 0.09
- link left_wrist_camera_link: geometry 
- link right_wrist_camera_link: geometry 

Commit message: New changes

File: rigby/urdf/rigby.urdf (robot description, URDF)
Before this commit: robot rigby, 40 links, 39 joints
Links:
- added link context_camera_2_link, mass 0.001; visual mesh filename=meshes/Oak-D.stl scale=0.001 0.001 0.001
- added link context_camera_2_optical_frame
Joints:
- added joint context_camera_2_joint: type fixed, parent base_link, child context_camera_2_link, origin xyz=0.186265 -0.000134 0.818559 rpy=0 -0.209731 0
- added joint context_camera_2_optical_joint: type fixed, parent context_camera_2_link, child context_camera_2_optical_frame, origin xyz=0 0 0 rpy=-1.5708 0 -1.5708
- joint context_camera_1_joint: origin xyz=0.079413 -0.005502 1.006560 rpy=0 0.48869 0 -> xyz=0.059988 -0.005502 1.016888 rpy=0 0.48869 0
